File: keyboard-pcb-first.sch (KiCad schematic (older format))
At the start: 24 parts, among them SW1 SW_Push, U1 ATmega32U4-AU, Y1 16MHz

Commit message: Started PCB
Parts:
- SW1: footprint (none) -> random-keyboard-parts:SKQG-1155865
Changed lines of the file:
@@
 F 0 "SW1" H 5000 2735 50  0000 C CNN
 F 1 "SW_Push" H 5000 2644 50  0000 C CNN
-F 2 "" H 5000 2650 50  0001 C CNN
+F 2 "random-keyboard-parts:SKQG-1155865" H 5000 2650 50  0001 C CNN
 F 3 "~" H 5000 2650 50  0001 C CNN
 	1    5000 2450
